File: PCB/2.5in-IDE-SSD.kicad_sch (KiCad schematic)
At the start: 91 parts, among them J1 Conn_02x22_Odd_Even, J2 Conn_02x02_Odd_Even, U1 SM2236, U2 TLV75533PDRV, U3 FlashBGA152, U4 FlashBGA152, U5 FlashBGA152, U6 FlashBGA152, U7 TLV75518PDRV

Commit message: Reversed state of master/slave select, making master mode enabled when jumper is removed
Parts:
- added Q1: PMBT2222AYS, Package_TO_SOT_SMD:SOT-363_SC-70-6, symbol Transistor_BJT:PMBT2222AYS
- added R27, R28: 10k, Resistor_SMD:R_0402_1005Metric, symbol Device:R_Small
- C1: LCSC (none) -> C15850
- C10, C11, C14, C15, C16, C17, C18, C19, C2, C20, C21, C22, C23, C24, C29, C30, C31, C32, C33, C34, C35, C36, C4, C6, C8: LCSC (none) -> C1525
- C12, C13, C41, C42: LCSC (none) -> C5673
- C25, C26, C27, C28, C37, C38, C39, C40: LCSC (none) -> C1691
- C3, C5, C7, C9: value 0.12uF -> 150nF; LCSC (none) -> C576725
- D1: LCSC (none) -> C5160703
- H1, H2, H3, H4, J1, J2, R17, R18, R19, R20, TP1, TP2, TP3, TP4, TP5, U1, U2, U7: now left out of the parts list
- R1, R10, R11, R12, R5, R6, R8, R9: LCSC (none) -> C163453
- R13: LCSC (none) -> C100044; now left out of the parts list
- R14: LCSC (none) -> C105875
- R15: value 300 -> 330; LCSC (none) -> C105875
- R16: LCSC (none) -> C60490
- R2, R3, R7: LCSC (none) -> C114765
- R21, R22, R23, R24: LCSC (none) -> C60488
- R25: LCSC (none) -> C100044
- R26: LCSC (none) -> C60485
- R4: LCSC (none) -> C60485; now left out of the parts list
- RN1, RN2, RN3, RN4: LCSC (none) -> C136851
- U3, U4, U5, U6: footprint Package_BGA:BGA-152_14x18mm_Layout13x17_P0.5mm -> cust:BGA-152_14x18mm_Layout13x17_P0.5mm; now left out of the parts list
Connections:
- net +3V3: now also R27.2, R28.2
- net GND: now also Q1.1 (E1), Q1.4 (E2)
- net HD_CSEL#: now also Q1.6 (C1); no longer J2.2 (Pin_2)
- net HD_CSEL_CONN#: now also Q1.5 (B2), R27.1; no longer J2.4 (Pin_4)
- new net: J2.2 (Pin_2), Q1.2 (B1), R28.1
- new net: J2.4 (Pin_4), Q1.3 (C2)
Other:
- note added: "No Jumper: Master 1-2 Short: Slave 2-4 Short: Cable Select"
- note removed: "1-2 Short: Master No Jumper: Slave 2-4 Short: Cable Select"
- moved on the sheet: J2
